File: 1.sch (KiCad schematic (older format))
At the start: 47 parts, among them J1 USB_B_Micro, J10 SPI2, J11 Micro_SD_Card, J12 Conn_01x04, J2 Power, J3 SWD, J4 Protected, J5 ADC, J6 SPI1, J7 UART1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

Commit message: op in windows
Parts:
- J1: symbol Connector:USB_B_Micro -> 1-rescue:USB_B_Micro-Connector
- J12: footprint Connector_PinSocket_2.54mm:PinSocket_1x03_P2.54mm_Vertical -> Connector_PinSocket_2.54mm:PinSocket_1x04_P2.54mm_Vertical; symbol Connector_Generic:Conn_01x03 -> Connector_Generic:Conn_01x04
- J4: footprint Connector_PinHeader_2.54mm:PinHeader_2x03_P2.54mm_Vertical -> Connector_PinSocket_2.54mm:PinSocket_2x03_P2.54mm_Vertical
- J9: value I2C2 -> Conn_01x04; footprint Connector_PinHeader_2.54mm:PinHeader_1x07_P2.54mm_Vertical -> Connector_PinSocket_2.54mm:PinSocket_1x07_P2.54mm_Vertical
Connections:
- wire segments 303 -> 302
Other:
- moved on the sheet: R10
Changed lines of the file:
@@
 F 0 "U1" H 6200 2561 50  0000 C CNN
 F 1 "STM32F103C8Tx" H 6200 2470 50  0000 C CNN
-F 2 "Package_QFP:LQFP-48_7x7mm_P0.5mm" H 5650 2750 50  0000 R CNN
+F 2 "Package_QFP:LQFP-48_7x7mm_P0.5mm" H 5650 2750 50  0001 R CNN
 F 3 "http://www.st.com/st-web-ui/static/active/en/resource/technical/document/datasheet/CD00161566.pdf" H 6250 4150 50  0001 C CNN
 	1    6250 4150
@@
 	0    -1   -1   0
 $EndComp
-Wire Wire Line
-	9450 2700 9350 2700
-Wire Wire Line
-	9450 2700 9450 2600
 $Comp
 L power:+3.3V #PWR0119
 U 1 1 609E08F0
-P 9450 2600
-F 0 "#PWR0119" H 9450 2450 50  0001 C CNN
-F 1 "+3.3V" H 9465 2773 50  0000 C CNN
-F 2 "" H 9450 2600 50  0001 C CNN
-F 3 "" H 9450 2600 50  0001 C CNN
-	1    9450 2600
+P 9450 2500
+F 0 "#PWR0119" H 9450 2350 50  0001 C CNN
+F 1 "+3.3V" H 9465 2673 50  0000 C CNN
+F 2 "" H 9450 2500 50  0001 C CNN
+F 3 "" H 9450 2500 50  0001 C CNN
+	1    9450 2500
 	-1   0    0    -1
-$EndComp
-$Comp
-L Connector_Generic:Conn_02x03_Odd_Even J4
-U 1 1 608D3B31
-P 9050 2800
-F 0 "J4" H 9100 3117 50  0000 C CNN
-F 1 "Protected" H 9100 3026 50  0000 C CNN
-F 2 "Connector_PinHeader_2.54mm:PinHeader_2x03_P2.54mm_Vertical" H 9050 2800 50  0001 C CNN
-F 3 "~" H 9050 2800 50  0001 C CNN
-	1    9050 2800
-	1    0    0    -1
 $EndComp
 $Comp
 L Connector_Generic:Conn_01x06 J6
 U 1 1 60955773
-P 9250 4550
-F 0 "J6" H 9330 4542 50  0000 L CNN
-F 1 "SPI1" H 9330 4451 50  0000 L CNN
-F 2 "Connector_PinHeader_2.54mm:PinHeader_1x06_P2.54mm_Vertical" H 9330 4405 50  0001 L CNN
-F 3 "~" H 9250 4550 50  0001 C CNN
-	1    9250 4550
-	1    0    0    -1
+P 9250 4650
+F 0 "J6" H 9330 4642 50  0000 L CNN
+F 1 "SPI1" H 9330 4551 50  0000 L CNN
+F 2 "Connector_PinHeader_2.54mm:PinHeader_1x06_P2.54mm_Vertical" H 9330 4505 50  0001 L CNN
+F 3 "~" H 9250 4650 50  0001 C CNN
+	1    9250 4650
+	1    0    0    1
 $EndComp
 Wire Wire Line
@@
 Wire Wire Line
 	8950 4250 8950 4350
-Wire Wire Line
-	8850 2700 8800 2700
 $Comp
 L Device:R R10
 U 1 1 61451B29
-P 8150 2800
-F 0 "R10" H 8220 2846 50  0000 L CNN
-F 1 "10k" H 8220 2755 50  0000 L CNN
-F 2 "Resistor_SMD:R_0603_1608Metric" V 8080 2800 50  0001 C CNN
-F 3 "~" H 8150 2800 50  0001 C CNN
-	1    8150 2800
+P 8150 2700
+F 0 "R10" H 8220 2746 50  0000 L CNN
+F 1 "10k" H 8220 2655 50  0000 L CNN
+F 2 "Resistor_SMD:R_0603_1608Metric" V 8080 2700 50  0001 C CNN
+F 3 "~" H 8150 2700 50  0001 C CNN
+	1    8150 2700
 	1    0    0    -1
 $EndComp
@@
 L power:GND #PWR0127
 U 1 1 61451B2F
-P 8150 3000
-F 0 "#PWR0127" H 8150 2750 50  0001 C CNN
-F 1 "GND" H 8155 2827 50  0000 C CNN
-F 2 "" H 8150 3000 50  0001 C CNN
-F 3 "" H 8150 3000 50  0001 C CNN
-	1    8150 3000
-	1    0    0    -1
-$EndComp
-Wire Wire Line
-	8150 2950 8150 3000
-Wire Wire Line
-	8150 2650 8150 2550
-Wire Wire Line
-	8150 2550 8800 2550
-Wire Wire Line
-	8800 2550 8800 2700
-Connection ~ 8800 2700
+P 8150 2900
+F 0 "#PWR0127" H 8150 2650 50  0001 C CNN
+F 1 "GND" H 8155 2727 50  0000 C CNN
+F 2 "" H 8150 2900 50  0001 C CNN
+F 3 "" H 8150 2900 50  0001 C CNN
+	1    8150 2900
+	1    0    0    -1
+$EndComp
+Wire Wire Line
+	8150 2850 8150 2900
+Wire Wire Line
+	8150 2550 8850 2550
+Wire Wire Line
+	8850 2550 8850 2700
 $Comp
 L Switch:SW_Push K3
@@
 	1    0    0    -1
 $EndComp
-$Comp
-L Connector:USB_B_Micro J1
-U 1 1 60B0F0BF
-P 6600 1250
-F 0 "J1" H 6657 1717 50  0000 C CNN
-F 1 "USB_B_Micro" H 6657 1626 50  0000 C CNN
-F 2 "Connector_USB:USB_Micro-B_GCT_USB3076-30-A" H 6750 1200 50  0001 C CNN
-F 3 "~" H 6750 1200 50  0001 C CNN
-	1    6600 1250
-	1    0    0    -1
-$EndComp
 Wire Wire Line
 	6900 1050 7500 1050
@@
 Wire Wire Line
 	3550 3700 3650 3700
-Wire Wire Line
-	3500 3600 3650 3600
 $Comp
 L Connector_Generic:Conn_02x06_Odd_Even J8
@@
 	1    0    0    -1
 $EndComp
-Wire Wire Line
-	3500 3500 3500 3600
-Connection ~ 3500 3600
 Connection ~ 3550 4100
-Wire Wire Line
-	3500 3600 3500 4000
 $Comp
 L power:GND #PWR0125
@@
 	4350 5250 4350 5300
 Wire Wire Line
-	4200 5100 4200 5300
-Connection ~ 4250 5000
-Wire Wire Line
 	4350 5000 4250 5000
 Wire Wire Line
@@
 	1    0    0    -1
 $EndComp
-Wire Wire Line
-	4150 5200 4300 5200
 Text HLabel 4300 5200 2    50   Input ~ 0
 PB2
 Connection ~ 4250 4600
-Wire Wire Line
-	4250 5000 4150 5000
 Wire Wire Line
 	4250 4600 4250 5000
@@
 	1    0    0    -1
 $EndComp
-Connection ~ 4200 5100
 $Comp
 L power:GND #PWR0128
@@
 Wire Wire Line
 	4200 4700 4150 4700
-Wire Wire Line
-	4200 5100 4200 4700
-Wire Wire Line
-	4150 5100 4200 5100
-$Comp
-L Connector_Generic:Conn_01x07 J9
-U 1 1 6153FBE5
-P 3950 4900
-F 0 "J9" H 3881 5396 50  0000 C CNN
-F 1 "I2C2" H 3881 5329 50  0000 C CNN
-F 2 "Connector_PinHeader_2.54mm:PinHeader_1x07_P2.54mm_Vertical" H 3950 4900 50  0001 C CNN
-F 3 "~" H 3950 4900 50  0001 C CNN
-	1    3950 4900
-	-1   0    0    -1
-$EndComp
 NoConn ~ 2500 6400
 NoConn ~ 2500 7100
@@
 Wire Wire Line
 	10150 2900 10600 2900
-Text Label 9700 2800 2    50   ~ 0
+Text Label 8500 2800 0    50   ~ 0
 SWCLK
 Wire Wire Line
-	9350 2800 9700 2800
+	8850 2800 8500 2800
 Text Label 8500 2700 0    50   ~ 0
 BOOT0
 Wire Wire Line
-	8500 2700 8800 2700
-Wire Wire Line
-	8500 2800 8850 2800
-Wire Wire Line
-	8500 2900 8850 2900
-Text Label 8500 2800 0    50   ~ 0
+	8500 2700 8850 2700
+Wire Wire Line
+	9700 2800 9350 2800
+Wire Wire Line
+	9700 2900 9350 2900
+Text Label 9700 2800 2    50   ~ 0
 SWDIO
+Text Label 9700 2900 2    50   ~ 0
+USB_D-
 Text Label 8500 2900 0    50   ~ 0
-USB_D-
-Text Label 9700 2900 2    50   ~ 0
 USB_D+
 Wire Wire Line
-	9350 2900 9700 2900
+	8850 2900 8500 2900
 Wire Wire Line
 	1000 2500 1000 2700
@@
 $EndComp
 $Comp
-L Connector_Generic:Conn_01x03 J12
+L Connector_Generic:Conn_01x04 J12
 U 1 1 609759C3
-P 9250 3500
-F 0 "J12" H 9330 3542 50  0000 L CNN
-F 1 "Conn_01x04" H 9330 3451 50  0000 L CNN
-F 2 "Connector_PinSocket_2.54mm:PinSocket_1x03_P2.54mm_Vertical" H 9250 3500 50  0001 C CNN
-F 3 "~" H 9250 3500 50  0001 C CNN
-	1    9250 3500
-	1    0    0    -1
-$EndComp
-Wire Wire Line
-	8950 3400 9050 3400
+P 9900 3700
+F 0 "J12" H 9980 3742 50  0000 L CNN
+F 1 "Conn_01x04" H 9980 3651 50  0000 L CNN
+F 2 "Connector_PinSocket_2.54mm:PinSocket_1x04_P2.54mm_Vertical" H 9900 3700 50  0001 C CNN
+F 3 "~" H 9900 3700 50  0001 C CNN
+	1    9900 3700
+	1    0    0    -1
+$EndComp
+Wire Wire Line
+	9600 3600 9700 3600
 $Comp
 L power:+3V3 #PWR0134
 U 1 1 6097B24C
-P 8950 3300
-F 0 "#PWR0134" H 8950 3150 50  0001 C CNN
-F 1 "+3V3" H 8965 3473 50  0000 C CNN
-F 2 "" H 8950 3300 50  0001 C CNN
-F 3 "" H 8950 3300 50  0001 C CNN
-	1    8950 3300
-	1    0    0    -1
-$EndComp
-Wire Wire Line
-	8950 3300 8950 3400
-Text Label 8750 3600 0    50   ~ 0
+P 9600 3500
+F 0 "#PWR0134" H 9600 3350 50  0001 C CNN
+F 1 "+3V3" H 9615 3673 50  0000 C CNN
+F 2 "" H 9600 3500 50  0001 C CNN
+F 3 "" H 9600 3500 50  0001 C CNN
+	1    9600 3500
+	1    0    0    -1
+$EndComp
+Wire Wire Line
+	9600 3500 9600 3600
+Text Label 9400 3800 0    50   ~ 0
 PA2
 Wire Wire Line
-	9050 3500 8950 3500
-Wire Wire Line
-	8950 3500 8950 3800
+	9700 3700 9600 3700
+Wire Wire Line
+	9600 3700 9600 4000
 $Comp
 L power:GND #PWR0135
 U 1 1 60995CA3
-P 8950 3800
-F 0 "#PWR0135" H 8950 3550 50  0001 C CNN
-F 1 "GND" H 8955 3627 50  0000 C CNN
-F 2 "" H 8950 3800 50  0001 C CNN
-F 3 "" H 8950 3800 50  0001 C CNN
-	1    8950 3800
-	1    0    0    -1
-$EndComp
-Wire Wire Line
-	8750 3600 9050 3600
+P 9600 4000
+F 0 "#PWR0135" H 9600 3750 50  0001 C CNN
+F 1 "GND" H 9605 3827 50  0000 C CNN
+F 2 "" H 9600 4000 50  0001 C CNN
+F 3 "" H 9600 4000 50  0001 C CNN
+	1    9600 4000
+	1    0    0    -1
+$EndComp
+Wire Wire Line
+	9400 3800 9700 3800
+Text Label 9400 3900 0    50   ~ 0
+PA3
+Wire Wire Line
+	9700 3900 9400 3900
+$Comp
+L 1-rescue:USB_B_Micro-Connector J1
+U 1 1 60B0F0BF
+P 6600 1250
+F 0 "J1" H 6657 1717 50  0000 C CNN
+F 1 "USB_B_Micro" H 6657 1626 50  0000 C CNN
+F 2 "Connector_USB:USB_Micro-B_GCT_USB3076-30-A" H 6750 1200 50  0001 C CNN
+F 3 "~" H 6750 1200 50  0001 C CNN
+	1    6600 1250
+	1    0    0    -1
+$EndComp
+$Comp
+L Connector_Generic:Conn_02x03_Odd_Even J4
+U 1 1 608D3B31
+P 9050 2800
+F 0 "J4" H 9100 3117 50  0000 C CNN
+F 1 "Protected" H 9100 3026 50  0000 C CNN
+F 2 "Connector_PinSocket_2.54mm:PinSocket_2x03_P2.54mm_Vertical" H 9050 2800 50  0001 C CNN
+F 3 "~" H 9050 2800 50  0001 C CNN
+	1    9050 2800
+	1    0    0    -1
+$EndComp
+Wire Wire Line
+	3500 3500 3500 3600
+Wire Wire Line
+	4200 4700 4200 5100
+$Comp
+L Connector_Generic:Conn_01x07 J9
+U 1 1 60BCC7ED
+P 3950 4900
+F 0 "J9" H 3868 5417 50  0000 C CNN
+F 1 "Conn_01x04" H 3868 5326 50  0000 C CNN
+F 2 "Connector_PinSocket_2.54mm:PinSocket_1x07_P2.54mm_Vertical" H 3950 4900 50  0001 C CNN
+F 3 "~" H 3950 4900 50  0001 C CNN
+	1    3950 4900
+	-1   0    0    -1
+$EndComp
+Wire Wire Line
+	4150 5000 4250 5000
+Connection ~ 4250 5000
+Wire Wire Line
+	4150 5100 4200 5100
+Connection ~ 4200 5100
+Wire Wire Line
+	4200 5100 4200 5300
+Wire Wire Line
+	4150 5200 4300 5200
+Wire Wire Line
+	3650 3600 3500 3600
+Connection ~ 3500 3600
+Wire Wire Line
+	3500 3600 3500 4000
+Connection ~ 8850 2700
+Wire Wire Line
+	9450 2500 9450 2700
+Wire Wire Line
+	9350 2700 9450 2700
 $EndSCHEMATC

Commit message: 改进
Parts:
- J1: symbol 1-rescue:USB_B_Micro-Connector -> 1-rescue:USB_B_Micro-Connector-1-rescue
Connections:
- wire segments 302 -> 304
Other:
- moved on the sheet: J4, R10
Changed lines of the file:
@@
 L power:+3.3V #PWR0119
 U 1 1 609E08F0
-P 9450 2500
-F 0 "#PWR0119" H 9450 2350 50  0001 C CNN
-F 1 "+3.3V" H 9465 2673 50  0000 C CNN
-F 2 "" H 9450 2500 50  0001 C CNN
-F 3 "" H 9450 2500 50  0001 C CNN
-	1    9450 2500
+P 7650 5400
+F 0 "#PWR0119" H 7650 5250 50  0001 C CNN
+F 1 "+3.3V" H 7665 5573 50  0000 C CNN
+F 2 "" H 7650 5400 50  0001 C CNN
+F 3 "" H 7650 5400 50  0001 C CNN
+	1    7650 5400
 	-1   0    0    -1
 $EndComp
@@
 L Device:R R10
 U 1 1 61451B29
-P 8150 2700
-F 0 "R10" H 8220 2746 50  0000 L CNN
-F 1 "10k" H 8220 2655 50  0000 L CNN
-F 2 "Resistor_SMD:R_0603_1608Metric" V 8080 2700 50  0001 C CNN
-F 3 "~" H 8150 2700 50  0001 C CNN
-	1    8150 2700
-	1    0    0    -1
+P 8900 5650
+F 0 "R10" H 8970 5696 50  0000 L CNN
+F 1 "10k" H 8970 5605 50  0000 L CNN
+F 2 "Resistor_SMD:R_0603_1608Metric" V 8830 5650 50  0001 C CNN
+F 3 "~" H 8900 5650 50  0001 C CNN
+	1    8900 5650
+	-1   0    0    -1
 $EndComp
 $Comp
 L power:GND #PWR0127
 U 1 1 61451B2F
-P 8150 2900
-F 0 "#PWR0127" H 8150 2650 50  0001 C CNN
-F 1 "GND" H 8155 2727 50  0000 C CNN
-F 2 "" H 8150 2900 50  0001 C CNN
-F 3 "" H 8150 2900 50  0001 C CNN
-	1    8150 2900
-	1    0    0    -1
-$EndComp
-Wire Wire Line
-	8150 2850 8150 2900
-Wire Wire Line
-	8150 2550 8850 2550
-Wire Wire Line
-	8850 2550 8850 2700
+P 8900 5850
+F 0 "#PWR0127" H 8900 5600 50  0001 C CNN
+F 1 "GND" H 8905 5677 50  0000 C CNN
+F 2 "" H 8900 5850 50  0001 C CNN
+F 3 "" H 8900 5850 50  0001 C CNN
+	1    8900 5850
+	-1   0    0    -1
+$EndComp
+Wire Wire Line
+	8900 5800 8900 5850
 $Comp
 L Switch:SW_Push K3
@@
 Wire Wire Line
 	10150 2900 10600 2900
-Text Label 8500 2800 0    50   ~ 0
+Text Label 7400 5700 0    50   ~ 0
 SWCLK
 Wire Wire Line
-	8850 2800 8500 2800
-Text Label 8500 2700 0    50   ~ 0
+	7750 5700 7400 5700
+Text Label 8600 5600 2    50   ~ 0
 BOOT0
 Wire Wire Line
-	8500 2700 8850 2700
-Wire Wire Line
-	9700 2800 9350 2800
-Wire Wire Line
-	9700 2900 9350 2900
-Text Label 9700 2800 2    50   ~ 0
+	8600 5700 8250 5700
+Wire Wire Line
+	8600 5800 8250 5800
+Text Label 8600 5700 2    50   ~ 0
 SWDIO
-Text Label 9700 2900 2    50   ~ 0
+Text Label 8600 5800 2    50   ~ 0
 USB_D-
-Text Label 8500 2900 0    50   ~ 0
+Text Label 7400 5800 0    50   ~ 0
 USB_D+
 Wire Wire Line
-	8850 2900 8500 2900
+	7750 5800 7400 5800
 Wire Wire Line
 	1000 2500 1000 2700
@@
 	9700 3900 9400 3900
 $Comp
-L 1-rescue:USB_B_Micro-Connector J1
+L 1-rescue:USB_B_Micro-Connector-1-rescue J1
 U 1 1 60B0F0BF
 P 6600 1250
@@
 F 3 "~" H 6750 1200 50  0001 C CNN
 	1    6600 1250
-	1    0    0    -1
-$EndComp
-$Comp
-L Connector_Generic:Conn_02x03_Odd_Even J4
-U 1 1 608D3B31
-P 9050 2800
-F 0 "J4" H 9100 3117 50  0000 C CNN
-F 1 "Protected" H 9100 3026 50  0000 C CNN
-F 2 "Connector_PinSocket_2.54mm:PinSocket_2x03_P2.54mm_Vertical" H 9050 2800 50  0001 C CNN
-F 3 "~" H 9050 2800 50  0001 C CNN
-	1    9050 2800
 	1    0    0    -1
 $EndComp
@@
 Wire Wire Line
 	3500 3600 3500 4000
-Connection ~ 8850 2700
-Wire Wire Line
-	9450 2500 9450 2700
-Wire Wire Line
-	9350 2700 9450 2700
+Wire Wire Line
+	7650 5400 7650 5600
+$Comp
+L Connector_Generic:Conn_02x03_Odd_Even J4
+U 1 1 608D3B31
+P 7950 5700
+F 0 "J4" H 8000 6017 50  0000 C CNN
+F 1 "Protected" H 8000 5926 50  0000 C CNN
+F 2 "Connector_PinSocket_2.54mm:PinSocket_2x03_P2.54mm_Vertical" H 7950 5700 50  0001 C CNN
+F 3 "~" H 7950 5700 50  0001 C CNN
+	1    7950 5700
+	1    0    0    -1
+$EndComp
+Wire Wire Line
+	8250 5600 8300 5600
+Wire Wire Line
+	8300 5600 8300 5400
+Wire Wire Line
+	8300 5400 8900 5400
+Wire Wire Line
+	8900 5400 8900 5500
+Connection ~ 8300 5600
+Wire Wire Line
+	8300 5600 8600 5600
+Wire Wire Line
+	7750 5600 7650 5600
 $EndSCHEMATC

Commit message: 重新布线，取消SWD和USB排针
Parts:
- removed J4: Protected, Connector_PinSocket_2.54mm:PinSocket_2x03_P2.54mm_Vertical, symbol Connector_Generic:Conn_02x03_Odd_Even
- added J?: Conn_01x02, symbol Connector_Generic:Conn_01x02
Connections:
- wire segments 304 -> 298
Other:
- moved on the sheet: R10
Changed lines of the file:
@@
 L Device:R R10
 U 1 1 61451B29
-P 8900 5650
-F 0 "R10" H 8970 5696 50  0000 L CNN
-F 1 "10k" H 8970 5605 50  0000 L CNN
-F 2 "Resistor_SMD:R_0603_1608Metric" V 8830 5650 50  0001 C CNN
-F 3 "~" H 8900 5650 50  0001 C CNN
-	1    8900 5650
+P 7650 5950
+F 0 "R10" H 7720 5996 50  0000 L CNN
+F 1 "10k" H 7720 5905 50  0000 L CNN
+F 2 "Resistor_SMD:R_0603_1608Metric" V 7580 5950 50  0001 C CNN
+F 3 "~" H 7650 5950 50  0001 C CNN
+	1    7650 5950
 	-1   0    0    -1
 $EndComp
@@
 L power:GND #PWR0127
 U 1 1 61451B2F
-P 8900 5850
-F 0 "#PWR0127" H 8900 5600 50  0001 C CNN
-F 1 "GND" H 8905 5677 50  0000 C CNN
-F 2 "" H 8900 5850 50  0001 C CNN
-F 3 "" H 8900 5850 50  0001 C CNN
-	1    8900 5850
+P 7650 6150
+F 0 "#PWR0127" H 7650 5900 50  0001 C CNN
+F 1 "GND" H 7655 5977 50  0000 C CNN
+F 2 "" H 7650 6150 50  0001 C CNN
+F 3 "" H 7650 6150 50  0001 C CNN
+	1    7650 6150
 	-1   0    0    -1
 $EndComp
 Wire Wire Line
-	8900 5800 8900 5850
+	7650 6100 7650 6150
 $Comp
 L Switch:SW_Push K3
@@
 Wire Wire Line
 	10150 2900 10600 2900
-Text Label 7400 5700 0    50   ~ 0
-SWCLK
-Wire Wire Line
-	7750 5700 7400 5700
-Text Label 8600 5600 2    50   ~ 0
+Text Label 7300 5700 0    50   ~ 0
 BOOT0
-Wire Wire Line
-	8600 5700 8250 5700
-Wire Wire Line
-	8600 5800 8250 5800
-Text Label 8600 5700 2    50   ~ 0
-SWDIO
-Text Label 8600 5800 2    50   ~ 0
-USB_D-
-Text Label 7400 5800 0    50   ~ 0
-USB_D+
-Wire Wire Line
-	7750 5800 7400 5800
 Wire Wire Line
 	1000 2500 1000 2700
@@
 Wire Wire Line
 	7650 5400 7650 5600
-$Comp
-L Connector_Generic:Conn_02x03_Odd_Even J4
-U 1 1 608D3B31
-P 7950 5700
-F 0 "J4" H 8000 6017 50  0000 C CNN
-F 1 "Protected" H 8000 5926 50  0000 C CNN
-F 2 "Connector_PinSocket_2.54mm:PinSocket_2x03_P2.54mm_Vertical" H 7950 5700 50  0001 C CNN
-F 3 "~" H 7950 5700 50  0001 C CNN
-	1    7950 5700
-	1    0    0    -1
-$EndComp
-Wire Wire Line
-	8250 5600 8300 5600
-Wire Wire Line
-	8300 5600 8300 5400
-Wire Wire Line
-	8300 5400 8900 5400
-Wire Wire Line
-	8900 5400 8900 5500
-Connection ~ 8300 5600
-Wire Wire Line
-	8300 5600 8600 5600
+Wire Wire Line
+	7650 5700 7650 5800
 Wire Wire Line
 	7750 5600 7650 5600
+$Comp
+L Connector_Generic:Conn_01x02 J?
+U 1 1 60B9BE52
+P 7950 5600
+F 0 "J?" H 8030 5592 50  0000 L CNN
+F 1 "Conn_01x02" H 8030 5501 50  0000 L CNN
+F 2 "" H 7950 5600 50  0001 C CNN
+F 3 "~" H 7950 5600 50  0001 C CNN
+	1    7950 5600
+	1    0    0    -1
+$EndComp
+Wire Wire Line
+	7750 5700 7650 5700
+Connection ~ 7650 5700
+Wire Wire Line
+	7650 5700 7300 5700
 $EndSCHEMATC

Commit message: add 104 caps
Parts:
- added C14, C15, C?: 104, Capacitor_SMD:C_0603_1608Metric, symbol Device:C_Small
- J4: renamed from J?; footprint (none) -> Connector_PinHeader_2.54mm:PinHeader_1x02_P2.54mm_Vertical
Connections:
- wire segments 298 -> 311
Other:
- moved on the sheet: C6
Changed lines of the file:
@@
 L Device:C_Small C6
 U 1 1 60A78AA2
-P 6950 2850
-F 0 "C6" H 7042 2896 50  0000 L CNN
-F 1 "104" H 7042 2805 50  0000 L CNN
-F 2 "Capacitor_SMD:C_0603_1608Metric" H 6950 2850 50  0001 C CNN
-F 3 "~" H 6950 2850 50  0001 C CNN
-	1    6950 2850
+P 6950 2800
+F 0 "C6" H 7042 2846 50  0000 L CNN
+F 1 "104" H 7042 2755 50  0000 L CNN
+F 2 "Capacitor_SMD:C_0603_1608Metric" H 6950 2800 50  0001 C CNN
+F 3 "~" H 6950 2800 50  0001 C CNN
+	1    6950 2800
 	1    0    0    -1
 $EndComp
@@
 L power:GND #PWR0133
 U 1 1 60A91FFF
-P 6950 3000
-F 0 "#PWR0133" H 6950 2750 50  0001 C CNN
-F 1 "GND" H 6955 2827 50  0000 C CNN
-F 2 "" H 6950 3000 50  0001 C CNN
-F 3 "" H 6950 3000 50  0001 C CNN
-	1    6950 3000
-	1    0    0    -1
-$EndComp
-Wire Wire Line
-	6950 2950 6950 3000
+P 6950 3050
+F 0 "#PWR0133" H 6950 2800 50  0001 C CNN
+F 1 "GND" H 6955 2877 50  0000 C CNN
+F 2 "" H 6950 3050 50  0001 C CNN
+F 3 "" H 6950 3050 50  0001 C CNN
+	1    6950 3050
+	1    0    0    -1
+$EndComp
+Wire Wire Line
+	6950 2900 6950 3000
 Wire Wire Line
 	6950 2600 6450 2600
 Wire Wire Line
-	6950 2600 6950 2750
+	6950 2600 6950 2700
 Connection ~ 6450 2600
 Wire Wire Line
@@
 	7750 5600 7650 5600
 $Comp
-L Connector_Generic:Conn_01x02 J?
+L Connector_Generic:Conn_01x02 J4
 U 1 1 60B9BE52
 P 7950 5600
-F 0 "J?" H 8030 5592 50  0000 L CNN
+F 0 "J4" H 8030 5592 50  0000 L CNN
 F 1 "Conn_01x02" H 8030 5501 50  0000 L CNN
-F 2 "" H 7950 5600 50  0001 C CNN
+F 2 "Connector_PinHeader_2.54mm:PinHeader_1x02_P2.54mm_Vertical" H 7950 5600 50  0001 C CNN
 F 3 "~" H 7950 5600 50  0001 C CNN
 	1    7950 5600
@@
 Wire Wire Line
 	7650 5700 7300 5700
+$Comp
+L Device:C_Small C14
+U 1 1 60D58B2E
+P 7250 2800
+F 0 "C14" H 7342 2846 50  0000 L CNN
+F 1 "104" H 7342 2755 50  0000 L CNN
+F 2 "Capacitor_SMD:C_0603_1608Metric" H 7250 2800 50  0001 C CNN
+F 3 "~" H 7250 2800 50  0001 C CNN
+	1    7250 2800
+	1    0    0    -1
+$EndComp
+$Comp
+L Device:C_Small C15
+U 1 1 60D711F0
+P 7550 2800
+F 0 "C15" H 7642 2846 50  0000 L CNN
+F 1 "104" H 7642 2755 50  0000 L CNN
+F 2 "Capacitor_SMD:C_0603_1608Metric" H 7550 2800 50  0001 C CNN
+F 3 "~" H 7550 2800 50  0001 C CNN
+	1    7550 2800
+	1    0    0    -1
+$EndComp
+Wire Wire Line
+	6950 2600 7250 2600
+Wire Wire Line
+	7250 2600 7250 2700
+Connection ~ 6950 2600
+Wire Wire Line
+	7250 2600 7550 2600
+Wire Wire Line
+	7550 2600 7550 2700
+Connection ~ 7250 2600
+Wire Wire Line
+	7250 2900 7250 3000
+Wire Wire Line
+	7250 3000 6950 3000
+Wire Wire Line
+	7550 2900 7550 3000
+Wire Wire Line
+	7550 3000 7250 3000
+Connection ~ 7250 3000
+Wire Wire Line
+	6950 3050 6950 3000
+Connection ~ 6950 3000
+$Comp
+L Device:C_Small C?
+U 1 1 60E609F1
+P 3200 3850
+F 0 "C?" H 3292 3896 50  0000 L CNN
+F 1 "104" H 3292 3805 50  0000 L CNN
+F 2 "Capacitor_SMD:C_0603_1608Metric" H 3200 3850 50  0001 C CNN
+F 3 "~" H 3200 3850 50  0001 C CNN
+	1    3200 3850
+	-1   0    0    -1
+$EndComp
+Wire Wire Line
+	3500 3600 3200 3600
+Wire Wire Line
+	3200 3600 3200 3750
+Wire Wire Line
+	3550 4100 3200 4100
+Wire Wire Line
+	3200 3950 3200 4100
 $EndSCHEMATC

Commit message: USB D+ 1.5k up res, 104 cap near SWD
Parts:
- added C?: 104, Capacitor_SMD:C_0603_1608Metric, symbol Device:C_Small
- added R?: 1.5k, Resistor_SMD:R_0603_1608Metric, symbol Device:R
- gave numbers to parts that had none: 1
Connections:
- wire segments 311 -> 318
Changed lines of the file:
@@
 Connection ~ 6450 2600
-Wire Wire Line
-	10400 2700 10600 2700
 Wire Wire Line
 	10400 2500 10400 2700
@@
 	1    0    0    1
 $EndComp
-Wire Wire Line
-	10600 3000 10600 3150
 $Comp
 L power:+5V #PWR0118
@@
 L power:GND #PWR0116
 U 1 1 60E0941E
-P 10600 3150
-F 0 "#PWR0116" H 10600 2900 50  0001 C CNN
-F 1 "GND" H 10605 2977 50  0000 C CNN
-F 2 "" H 10600 3150 50  0001 C CNN
-F 3 "" H 10600 3150 50  0001 C CNN
-	1    10600 3150
+P 10600 3250
+F 0 "#PWR0116" H 10600 3000 50  0001 C CNN
+F 1 "GND" H 10605 3077 50  0000 C CNN
+F 2 "" H 10600 3250 50  0001 C CNN
+F 3 "" H 10600 3250 50  0001 C CNN
+	1    10600 3250
 	1    0    0    -1
 $EndComp
@@
 USB_D-
 Wire Wire Line
-	6900 1250 7300 1250
+	6900 1250 7000 1250
 Wire Wire Line
 	6900 1350 7300 1350
@@
 SWDIO
 Wire Wire Line
-	10150 2800 10600 2800
-Wire Wire Line
 	10150 2900 10600 2900
 Text Label 7300 5700 0    50   ~ 0
@@
 Connection ~ 6950 3000
 $Comp
-L Device:C_Small C?
+L Device:C_Small C16
 U 1 1 60E609F1
 P 3200 3850
-F 0 "C?" H 3292 3896 50  0000 L CNN
+F 0 "C16" H 3292 3896 50  0000 L CNN
 F 1 "104" H 3292 3805 50  0000 L CNN
 F 2 "Capacitor_SMD:C_0603_1608Metric" H 3200 3850 50  0001 C CNN
@@
 Wire Wire Line
 	3200 3950 3200 4100
+$Comp
+L Device:R R?
+U 1 1 60F54872
+P 7000 1000
+F 0 "R?" H 7070 1046 50  0000 L CNN
+F 1 "1.5k" H 7070 955 50  0000 L CNN
+F 2 "Resistor_SMD:R_0603_1608Metric" V 6930 1000 50  0001 C CNN
+F 3 "~" H 7000 1000 50  0001 C CNN
+	1    7000 1000
+	1    0    0    -1
+$EndComp
+Wire Wire Line
+	7000 1150 7000 1250
+Connection ~ 7000 1250
+Wire Wire Line
+	7000 1250 7300 1250
+$Comp
+L power:+3V3 #PWR?
+U 1 1 60F7073C
+P 7000 750
+F 0 "#PWR?" H 7000 600 50  0001 C CNN
+F 1 "+3V3" H 7015 923 50  0000 C CNN
+F 2 "" H 7000 750 50  0001 C CNN
+F 3 "" H 7000 750 50  0001 C CNN
+	1    7000 750
+	1    0    0    -1
+$EndComp
+Wire Wire Line
+	7000 750  7000 850
+Wire Wire Line
+	10150 2800 10600 2800
+Wire Wire Line
+	10400 3050 10400 3150
+$Comp
+L Device:C_Small C?
+U 1 1 60FAC932
+P 10400 2950
+F 0 "C?" H 10492 2996 50  0000 L CNN
+F 1 "104" H 10492 2905 50  0000 L CNN
+F 2 "Capacitor_SMD:C_0603_1608Metric" H 10400 2950 50  0001 C CNN
+F 3 "~" H 10400 2950 50  0001 C CNN
+	1    10400 2950
+	-1   0    0    -1
+$EndComp
+Wire Wire Line
+	10600 3000 10600 3150
+Wire Wire Line
+	10400 2850 10400 2700
+Connection ~ 10400 2700
+Wire Wire Line
+	10400 2700 10600 2700
+Wire Wire Line
+	10400 3150 10600 3150
+Connection ~ 10600 3150
+Wire Wire Line
+	10600 3150 10600 3250
 $EndSCHEMATC
