File: 1.sch (KiCad schematic (older format))
At the start: 52 parts, among them J1 USB_B_Micro, J10 SPI2, J11 Micro_SD_Card, J12 Conn_01x04, J2 Power, J3 SWD, J4 Conn_01x02, J5 ADC, J6 SPI1, J7 UART1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

Commit message: save .sch file
Parts:
- gave numbers to parts that had none: 2
Changed lines of the file:
@@
 	3200 3950 3200 4100
 $Comp
-L Device:R R?
+L Device:R R12
 U 1 1 60F54872
 P 7000 1000
-F 0 "R?" H 7070 1046 50  0000 L CNN
+F 0 "R12" H 7070 1046 50  0000 L CNN
 F 1 "1.5k" H 7070 955 50  0000 L CNN
 F 2 "Resistor_SMD:R_0603_1608Metric" V 6930 1000 50  0001 C CNN
@@
 	7000 1250 7300 1250
 $Comp
-L power:+3V3 #PWR?
+L power:+3V3 #PWR0136
 U 1 1 60F7073C
 P 7000 750
-F 0 "#PWR?" H 7000 600 50  0001 C CNN
+F 0 "#PWR0136" H 7000 600 50  0001 C CNN
 F 1 "+3V3" H 7015 923 50  0000 C CNN
 F 2 "" H 7000 750 50  0001 C CNN
@@
 	10400 3050 10400 3150
 $Comp
-L Device:C_Small C?
+L Device:C_Small C17
 U 1 1 60FAC932
 P 10400 2950
-F 0 "C?" H 10492 2996 50  0000 L CNN
+F 0 "C17" H 10492 2996 50  0000 L CNN
 F 1 "104" H 10492 2905 50  0000 L CNN
 F 2 "Capacitor_SMD:C_0603_1608Metric" H 10400 2950 50  0001 C CNN

Commit message: PC13 replace I2C1 one of 3V3
Connections:
- wire segments 318 -> 317
Changed lines of the file:
@@
 	3550 4100 3650 4100
-Wire Wire Line
-	3500 4000 3650 4000
 Wire Wire Line
 	3550 3700 3650 3700
@@
 Connection ~ 3500 3600
 Wire Wire Line
-	3500 3600 3500 4000
-Wire Wire Line
 	7650 5400 7650 5600
 Wire Wire Line
@@
 Wire Wire Line
 	10600 3150 10600 3250
+Text Label 3300 4000 0    50   ~ 0
+RG_LED
+Wire Wire Line
+	3650 4000 3300 4000
 $EndSCHEMATC

Commit message: copy from windows, 成功打样
Parts:
- J4: value Conn_01x02 -> Conn_01x03; footprint Connector_PinHeader_2.54mm:PinHeader_1x02_P2.54mm_Vertical -> Connector_PinHeader_2.54mm:PinHeader_1x03_P2.54mm_Vertical; symbol Connector_Generic:Conn_01x02 -> Connector_Generic:Conn_01x03
Connections:
- wire segments 317 -> 319
Other:
- moved on the sheet: R10
Changed lines of the file:
@@
-$EndComp
-$Comp
-L power:+3.3V #PWR0119
-U 1 1 609E08F0
-P 7650 5400
-F 0 "#PWR0119" H 7650 5250 50  0001 C CNN
-F 1 "+3.3V" H 7665 5573 50  0000 C CNN
-F 2 "" H 7650 5400 50  0001 C CNN
-F 3 "" H 7650 5400 50  0001 C CNN
-	1    7650 5400
-	-1   0    0    -1
 $EndComp
 $Comp
@@
 L Device:R R10
 U 1 1 61451B29
-P 7650 5950
-F 0 "R10" H 7720 5996 50  0000 L CNN
-F 1 "10k" H 7720 5905 50  0000 L CNN
-F 2 "Resistor_SMD:R_0603_1608Metric" V 7580 5950 50  0001 C CNN
-F 3 "~" H 7650 5950 50  0001 C CNN
-	1    7650 5950
+P 7700 6050
+F 0 "R10" H 7770 6096 50  0000 L CNN
+F 1 "10k" H 7770 6005 50  0000 L CNN
+F 2 "Resistor_SMD:R_0603_1608Metric" V 7630 6050 50  0001 C CNN
+F 3 "~" H 7700 6050 50  0001 C CNN
+	1    7700 6050
 	-1   0    0    -1
 $EndComp
@@
 L power:GND #PWR0127
 U 1 1 61451B2F
-P 7650 6150
-F 0 "#PWR0127" H 7650 5900 50  0001 C CNN
-F 1 "GND" H 7655 5977 50  0000 C CNN
-F 2 "" H 7650 6150 50  0001 C CNN
-F 3 "" H 7650 6150 50  0001 C CNN
-	1    7650 6150
+P 7700 6250
+F 0 "#PWR0127" H 7700 6000 50  0001 C CNN
+F 1 "GND" H 7705 6077 50  0000 C CNN
+F 2 "" H 7700 6250 50  0001 C CNN
+F 3 "" H 7700 6250 50  0001 C CNN
+	1    7700 6250
 	-1   0    0    -1
 $EndComp
 Wire Wire Line
-	7650 6100 7650 6150
+	7700 6200 7700 6250
 $Comp
 L Switch:SW_Push K3
@@
 Wire Wire Line
 	10150 2900 10600 2900
-Text Label 7300 5700 0    50   ~ 0
+Text Label 7350 5700 0    50   ~ 0
 BOOT0
 Wire Wire Line
@@
 Connection ~ 3500 3600
 Wire Wire Line
-	7650 5400 7650 5600
-Wire Wire Line
-	7650 5700 7650 5800
-Wire Wire Line
-	7750 5600 7650 5600
-$Comp
-L Connector_Generic:Conn_01x02 J4
-U 1 1 60B9BE52
-P 7950 5600
-F 0 "J4" H 8030 5592 50  0000 L CNN
-F 1 "Conn_01x02" H 8030 5501 50  0000 L CNN
-F 2 "Connector_PinHeader_2.54mm:PinHeader_1x02_P2.54mm_Vertical" H 7950 5600 50  0001 C CNN
-F 3 "~" H 7950 5600 50  0001 C CNN
-	1    7950 5600
-	1    0    0    -1
-$EndComp
-Wire Wire Line
-	7750 5700 7650 5700
-Connection ~ 7650 5700
-Wire Wire Line
-	7650 5700 7300 5700
+	7850 5700 7700 5700
+Connection ~ 7700 5700
+Wire Wire Line
+	7700 5700 7350 5700
 $Comp
 L Device:C_Small C14
@@
 Wire Wire Line
 	10600 3150 10600 3250
-Text Label 3300 4000 0    50   ~ 0
+Wire Wire Line
+	3650 4000 3500 4000
+Wire Wire Line
+	3500 4000 3500 3600
+Text Label 7350 5800 0    50   ~ 0
 RG_LED
 Wire Wire Line
-	3650 4000 3300 4000
+	7700 5450 7700 5600
+$Comp
+L power:+3.3V #PWR0119
+U 1 1 609E08F0
+P 7700 5450
+F 0 "#PWR0119" H 7700 5300 50  0001 C CNN
+F 1 "+3.3V" H 7715 5623 50  0000 C CNN
+F 2 "" H 7700 5450 50  0001 C CNN
+F 3 "" H 7700 5450 50  0001 C CNN
+	1    7700 5450
+	-1   0    0    -1
+$EndComp
+Wire Wire Line
+	7850 5600 7700 5600
+$Comp
+L Connector_Generic:Conn_01x03 J4
+U 1 1 60B9BE52
+P 8050 5700
+F 0 "J4" H 8130 5692 50  0000 L CNN
+F 1 "Conn_01x03" H 8130 5601 50  0000 L CNN
+F 2 "Connector_PinHeader_2.54mm:PinHeader_1x03_P2.54mm_Vertical" H 8050 5700 50  0001 C CNN
+F 3 "~" H 8050 5700 50  0001 C CNN
+	1    8050 5700
+	1    0    0    -1
+$EndComp
+Wire Wire Line
+	7700 5700 7700 5900
+Wire Wire Line
+	7350 5800 7850 5800
 $EndSCHEMATC
